Commit message: chnage name of gripper link from arm_gripper link

File: p_rob_description/urdf/p_rob.transmission.xacro (robot description, xacro)
@@ -62,11 +62,11 @@
 		</actuator>
 	</transmission>
-	<transmission name="${prefix}gripper_trans">
+	<transmission name="gripper_trans">
 		<type>transmission_interface/SimpleTransmission</type>
-		<joint name="${prefix}gripper">
+		<joint name="gripper">
 			<hardwareInterface>PositionJointInterface</hardwareInterface>
 			<hardwareInterface>VelocityJointInterface</hardwareInterface>
 		</joint>
-		<actuator name="${prefix}gripper_motor">
+		<actuator name="gripper_motor">
 			<mechanicalReduction>1</mechanicalReduction>
 		</actuator>
